File: touch.brd (EAGLE design)
At the start: 91.4 x 50.5 mm, 25 parts, among them IC1 MAX203ECWP, IC2 PIC18F14Q41-I_SO, X1 22-23-2021

Commit message: up
Parts:
- added C7: 10uf, rcl:C0805
- added F1: 0.75A, polyfuse-smd_10:1206L
- added L1: 1000, inductor-neosid:SM-1206
- C1, C4: value (none) -> 10uf
- C2, C3, C5, C6: value (none) -> 0.1
- D1: value (none) -> 5.6V
- R1, R2: value (none) -> 56
- R3: value (none) -> 10K
- R4: value (none) -> 1k
- R5: value (none) -> 200
Connections:
- new net N$16: F1.2, X1.1
- new net N$20: F1.1, L1.1
- net GND: now also C7.2
- net VCC: now also C7.1, L1.2; no longer X1.1
Routing:
- net VCC: track 133.6 -> 155.7 mm, vias 2 -> 0
- net GND: track 19.5 -> 0.70 mm, vias 1 -> 0
- net N$16: track 0.00 -> 8.43 mm
- net TX1: track 54.6 -> 62.4 mm, vias 3 -> 0
- net N$20: track 0.00 -> 3.30 mm
- net N$8: track 54.7 -> 51.5 mm
- net N$13: track 31.9 -> 29.9 mm, vias 0 -> 1
- net TX2: track 13.6 -> 11.9 mm
- net N$18: track 19.7 -> 18.2 mm
- net N$15: track 28.7 -> 29.2 mm, vias 0 -> 1
- net N$10: track 31.4 -> 31.1 mm, vias 0 -> 1
- net N$9: track 48.2 -> 48.5 mm, vias 0 -> 2
- added copper zone on layer 16, net GND

Commit message: up
Parts:
- added LED_MODE: RED, led:CHIPLED_0805
- added LED_POWER: GREEN, led:CHIPLED_0805
- added R6, R7: 200, rcl:R0805
- added SV2: (no value), con-lstb:MA04-2
- added SV3: (no value), con-lstb:MA03-2
Connections:
- removed net N$17: C5.1, R2.1, R3.1, S1.1, S1.2
- new net CS: IC2.11, SV2.6
- new net MIN0: IC2.16, SV2.1
- new net MIN1: IC2.7, SV2.3
- new net MISC: IC2.10, SV3.3
- new net MISO: IC2.13, SV2.7
- new net MLED: IC2.6, R7.2
- new net MOSI: IC2.17, SV2.5
- new net N$21: LED_POWER.A, R6.1
- new net N$22: LED_MODE.A, R7.1
- new net RELAY: IC2.9, SV3.1
- new net RLED: IC2.5, R4.1
- new net SCK: IC2.3, SV2.8
- new net SMCLEAR: C5.1, R2.1, R3.1, S1.1, S1.2, SV3.5
- net GND: now also LED_MODE.C, LED_POWER.C, SV2.2, SV2.4, SV3.2
- net VCC: now also R6.2; no longer R4.1
Routing:
- net SMCLEAR: track 0.00 -> 72.1 mm, vias 0 -> 2
- net MISO: track 0.00 -> 56.2 mm, vias 0 -> 2
- net RELAY: track 0.00 -> 55.1 mm, vias 0 -> 1
- net MIN0: track 0.00 -> 53.7 mm, vias 0 -> 2
- net MISC: track 0.00 -> 51.8 mm, vias 0 -> 1
- net MIN1: track 0.00 -> 50.9 mm, vias 0 -> 2
- net CS: track 0.00 -> 50.8 mm, vias 0 -> 2
- net MLED: track 0.00 -> 49.9 mm, vias 0 -> 2
- net SCK: track 0.00 -> 49.1 mm, vias 0 -> 1
- net MOSI: track 0.00 -> 49.1 mm, vias 0 -> 1
- net N$17: track 41.7 -> 0.00 mm, vias 2 -> 0
- net VCC: track 155.7 -> 192.8 mm
- net RLED: track 0.00 -> 32.0 mm
- net GND: track 0.70 -> 18.1 mm, vias 0 -> 1
- net N$22: track 0.00 -> 15.6 mm
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
Commit message: up
Parts:
- added TTLRS232: (no value), con-lstb:MA05-1
- renumbered SV1 to ICSP, SV2 to DIO2/SPI, SV3 to DIO3, X1 to POWER
Connections:
- net CLKIN: now also DIO3.4
- net GND: now also TTLRS232.1
- net RX1: now also TTLRS232.2
- net RX2: now also TTLRS232.4
- net TX1: now also TTLRS232.3
- net TX2: now also TTLRS232.5
- net VCC: now also DIO3.6
Routing:
- net CLKIN: track 10.6 -> 53.2 mm, vias 0 -> 1
- net MLED: track 49.9 -> 92.0 mm, vias 2 -> 0
- net N$8: track 51.5 -> 93.0 mm, vias 2 -> 0
- net N$9: track 48.8 -> 80.7 mm, vias 2 -> 0
- net RLED: track 32.0 -> 47.4 mm
- net GND: track 18.1 -> 3.45 mm, vias 1 -> 3
- net CS: track 50.8 -> 36.9 mm, vias 2 -> 1
- net MISO: track 56.2 -> 42.6 mm, vias 2 -> 1
- net N$14: track 8.28 -> 21.5 mm
- net SCK: track 49.1 -> 61.1 mm
- net N$11: track 38.1 -> 49.4 mm, vias 2 -> 0
- net TX1: track 62.7 -> 54.9 mm, vias 0 -> 3
- net RX2: track 21.2 -> 27.6 mm
- net N$2: track 22.6 -> 17.0 mm, vias 0 -> 1
- net SMCLEAR: track 72.1 -> 67.1 mm
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
Commit message: up
Routing:
- net GND: track 3.45 -> 27.0 mm, vias 3 -> 7
- net VCC: track 190.8 -> 214.3 mm, vias 8 -> 7
- net RLED: track 47.4 -> 25.1 mm
- net MLED: track 92.0 -> 71.0 mm
- net N$8: track 93.0 -> 78.6 mm
- net SCK: track 61.1 -> 48.0 mm
- net N$14: track 21.5 -> 9.28 mm
- net SMCLEAR: track 67.1 -> 77.8 mm, vias 2 -> 1
- net RX2: track 27.6 -> 20.7 mm
- net MIN1: track 46.9 -> 43.3 mm
- net N$1: track 17.9 -> 15.0 mm
- net N$2: track 17.0 -> 19.7 mm
- net N$9: track 80.7 -> 83.3 mm
- net N$11: track 49.4 -> 47.2 mm
- net MOSI: track 51.1 -> 49.1 mm
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Other:
- board text added: "Q41 vtouch 1.0"

Commit message: up
Connections:
- net GND: now also HOST_PORT1.5, ICSP.3; no longer HOST_PORT1.1, ICSP.2
- net VCC: now also ICSP.2; no longer ICSP.3
Other:
- board text added: "Q41 vtouch 1.1"
- board text removed: "Q41 vtouch 1.0"
Changed lines of the file:
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@@
 <hole x="87.63" y="3.81" drill="1"/>
 <hole x="87.63" y="46.99" drill="1"/>
-<text x="71.12" y="5.08" size="1.778" layer="1" font="vector" ratio="15">Q41 vtouch 1.0</text>
+<text x="71.12" y="5.08" size="1.778" layer="1" font="vector" ratio="15">Q41 vtouch 1.1</text>
 </plain>
 <attributes>
@@
 <autorouter>
 <pass name="Default">
-<param name="RoutingGrid" value="3mil"/>
+<param name="RoutingGrid" value="6.25mil"/>
 <param name="AutoGrid" value="1"/>
 <param name="Efforts" value="2"/>
 <param name="TopRouterVariant" value="1"/>
 <param name="tpViaShape" value="round"/>
-<param name="PrefDir.1" value="a"/>
-<param name="PrefDir.2" value="a"/>
+<param name="PrefDir.1" value="*"/>
+<param name="PrefDir.2" value="*"/>
 <param name="PrefDir.3" value="0"/>
 <param name="PrefDir.4" value="0"/>
@@
 <param name="PrefDir.13" value="0"/>
 <param name="PrefDir.14" value="0"/>
-<param name="PrefDir.15" value="a"/>
-<param name="PrefDir.16" value="a"/>
+<param name="PrefDir.15" value="*"/>
+<param name="PrefDir.16" value="-"/>
 <param name="cfVia" value="1"/>
 <param name="cfNonPref" value="5"/>
@@
 <contactref element="HOST_PORT1" pad="MH1"/>
 <contactref element="SCREEN_PORT2" pad="5"/>
-<contactref element="HOST_PORT1" pad="1"/>
 <contactref element="C3" pad="2"/>
 <contactref element="C4" pad="2"/>
@@
 <contactref element="C1" pad="2"/>
 <contactref element="IC2" pad="20"/>
-<contactref element="ICSP" pad="2"/>
 <contactref element="C5" pad="2"/>
 <polygon width="0.1524" layer="1">
@@
 <wire x1="80.23" y1="41.69" x2="80.01" y2="41.91" width="0.3048" layer="1"/>
 <wire x1="80.01" y1="41.91" x2="75.565" y2="37.465" width="0.3048" layer="1"/>
+<contactref element="ICSP" pad="3"/>
+<contactref element="HOST_PORT1" pad="5"/>
 </signal>
 <signal name="VCC" class="1">
@@
 <contactref element="C4" pad="1"/>
 <contactref element="D1" pad="C"/>
-<contactref element="ICSP" pad="3"/>
 <contactref element="R3" pad="2"/>
 <contactref element="OS1" pad="4"/>
@@
 <wire x1="86.1822" y1="10.9728" x2="86.1822" y2="11.5062" width="0.3048" layer="2"/>
 <wire x1="80.0862" y1="4.8768" x2="86.1822" y2="10.9728" width="0.3048" layer="2"/>
-<wire x1="60.8076" y1="4.8768" x2="80.0862" y2="4.8768" width="0.3048" layer="2"/>
-<wire x1="59.7408" y1="3.81" x2="60.8076" y2="4.8768" width="0.3048" layer="2"/>
-<wire x1="59.7408" y1="3.81" x2="59.69" y2="3.81" width="0.3048" layer="2"/>
+<wire x1="59.2074" y1="4.8768" x2="80.0862" y2="4.8768" width="0.3048" layer="2"/>
 <wire x1="46.3296" y1="27.6606" x2="46.3296" y2="29.2608" width="0.3048" layer="1"/>
 <wire x1="46.3296" y1="26.289" x2="46.3296" y2="27.6606" width="0.3048" layer="2"/>
@@
 <wire x1="49.0728" y1="4.8768" x2="44.9961" y2="8.9535" width="0.3048" layer="2"/>
 <wire x1="44.9961" y1="8.9535" x2="41.2242" y2="12.7254" width="0.3048" layer="2"/>
-<wire x1="58.5978" y1="4.8768" x2="49.0728" y2="4.8768" width="0.3048" layer="2"/>
-<wire x1="59.5884" y1="3.8862" x2="58.5978" y2="4.8768" width="0.3048" layer="2"/>
 <wire x1="46.3296" y1="29.2608" x2="46.355" y2="29.2608" width="0.3048" layer="1"/>
-<wire x1="59.5884" y1="3.8862" x2="59.69" y2="3.81" width="0.3048" layer="2"/>
 <wire x1="30.861" y1="43.9674" x2="30.861" y2="45.72" width="0.3048" layer="1"/>
 <wire x1="30.861" y1="43.1292" x2="30.861" y2="43.9674" width="0.3048" layer="2"/>
@@
 <via x="44.958" y="8.9154" extent="1-16" drill="0.35"/>
 <via x="39.0906" y="15.4686" extent="1-16" drill="0.35"/>
+<contactref element="ICSP" pad="2"/>
+<wire x1="58.1406" y1="3.81" x2="57.15" y2="3.81" width="0.3048" layer="2"/>
+<wire x1="59.2074" y1="4.8768" x2="58.1406" y2="3.81" width="0.3048" layer="2"/>
+<wire x1="56.0832" y1="3.8862" x2="57.0738" y2="3.8862" width="0.3048" layer="2"/>
+<wire x1="55.0926" y1="4.8768" x2="56.0832" y2="3.8862" width="0.3048" layer="2"/>
+<wire x1="49.0728" y1="4.8768" x2="55.0926" y2="4.8768" width="0.3048" layer="2"/>
+<wire x1="57.0738" y1="3.8862" x2="57.15" y2="3.81" width="0.3048" layer="2"/>
 </signal>
 <signal name="N$1">

Commit message: up
Parts:
- removed LED_MODE: RED, led:CHIPLED_0805
- removed LED_POWER: GREEN, led:CHIPLED_0805
- added GLORY: 22-23-2021, con-molex:22-23-2021
- added MODE, PWR: Green, led:CHIPLED_1206
- R4: value 1k -> 1.2k
- R6, R7: value 200 -> 1.2k
Connections:
- net N$10 renamed DB1
- net N$13 renamed DB0
- net N$15 renamed PGM
- removed net N$22: LED_MODE.A, R7.1
- new net N$17: MODE.A, R7.1
- net GND: now also MODE.C, PWR.C; no longer LED_MODE.C, LED_POWER.C
- net N$21: now also PWR.A; no longer LED_POWER.A
- net VCC: now also GLORY.1, GLORY.2
Routing:
- net N$22: track 15.6 -> 0.00 mm
- net N$17: track 0.00 -> 12.3 mm
- net GND: track 27.0 -> 15.7 mm, vias 7 -> 20
- net VCC: track 214.3 -> 222.3 mm
- net MLED: track 71.0 -> 72.8 mm
- net SMCLEAR: track 77.8 -> 79.5 mm
- net N$21: track 3.61 -> 4.20 mm

Commit message: up
Routing:
- net N$9: track 83.3 -> 69.1 mm, vias 0 -> 2
Changed lines of the file:
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@@
 <param name="RoutingGrid" value="6.25mil"/>
 <param name="AutoGrid" value="1"/>
-<param name="Efforts" value="2"/>
+<param name="Efforts" value="0"/>
 <param name="TopRouterVariant" value="1"/>
 <param name="tpViaShape" value="round"/>
@@
 <contactref element="IC2" pad="20"/>
 <contactref element="C5" pad="2"/>
-<polygon width="0.1524" layer="1">
+<polygon width="0.1524" layer="1" rank="6">
 <vertex x="10.16" y="48.26"/>
 <vertex x="10.16" y="7.62"/>
@@
 <wire x1="7.8486" y1="25.6032" x2="7.9248" y2="25.6032" width="0.1524" layer="1"/>
 <wire x1="7.62" y1="25.6032" x2="7.62" y2="25.654" width="0.1524" layer="1"/>
-<wire x1="42.5958" y1="32.9946" x2="42.5958" y2="29.2608" width="0.1524" layer="1"/>
-<wire x1="37.8714" y1="37.719" x2="42.5958" y2="32.9946" width="0.1524" layer="1"/>
-<wire x1="37.8714" y1="48.5394" x2="37.8714" y2="37.719" width="0.1524" layer="1"/>
-<wire x1="37.0332" y1="49.3776" x2="37.8714" y2="48.5394" width="0.1524" layer="1"/>
-<wire x1="9.6774" y1="49.3776" x2="37.0332" y2="49.3776" width="0.1524" layer="1"/>
-<wire x1="8.6106" y1="48.3108" x2="9.6774" y2="49.3776" width="0.1524" layer="1"/>
-<wire x1="8.6106" y1="34.2138" x2="8.6106" y2="48.3108" width="0.1524" layer="1"/>
-<wire x1="7.8486" y1="33.4518" x2="8.6106" y2="34.2138" width="0.1524" layer="1"/>
-<wire x1="7.8486" y1="25.6032" x2="7.8486" y2="33.4518" width="0.1524" layer="1"/>
-<wire x1="42.5958" y1="29.2608" x2="42.545" y2="29.2608" width="0.1524" layer="1"/>
 <wire x1="7.8486" y1="25.6032" x2="7.62" y2="25.654" width="0.1524" layer="1"/>
+<wire x1="42.545" y1="31.115" x2="42.545" y2="29.2608" width="0.1524" layer="1"/>
+<wire x1="41.275" y1="32.385" x2="42.545" y2="31.115" width="0.1524" layer="1"/>
+<wire x1="38.1" y1="32.385" x2="41.275" y2="32.385" width="0.1524" layer="1"/>
+<wire x1="36.195" y1="30.48" x2="38.1" y2="32.385" width="0.1524" layer="1"/>
+<wire x1="36.195" y1="26.67" x2="36.195" y2="30.48" width="0.1524" layer="1"/>
+<wire x1="35.56" y1="26.035" x2="36.195" y2="26.67" width="0.1524" layer="1"/>
+<via x="34.29" y="25.4" extent="1-16" drill="0.35"/>
+<wire x1="34.29" y1="25.4" x2="34.925" y2="26.035" width="0.1524" layer="1"/>
+<wire x1="34.925" y1="26.035" x2="35.56" y2="26.035" width="0.1524" layer="1"/>
+<wire x1="31.75" y1="25.4" x2="24.13" y2="33.02" width="0.1524" layer="2"/>
+<wire x1="24.13" y1="33.02" x2="24.13" y2="35.56" width="0.1524" layer="2"/>
+<wire x1="5.3594" y1="33.430325" x2="5.3594" y2="32.609675" width="0.1524" layer="2"/>
+<wire x1="5.3594" y1="32.609675" x2="6.269875" y2="31.6992" width="0.1524" layer="2"/>
+<wire x1="6.269875" y1="31.6992" x2="6.531725" y2="31.6992" width="0.1524" layer="2"/>
+<wire x1="6.531725" y1="31.6992" x2="7.62" y2="30.610925" width="0.1524" layer="2"/>
+<wire x1="7.489075" y1="35.56" x2="5.3594" y2="33.430325" width="0.1524" layer="2"/>
+<wire x1="34.29" y1="25.4" x2="31.75" y2="25.4" width="0.1524" layer="2"/>
+<wire x1="24.13" y1="35.56" x2="7.489075" y2="35.56" width="0.1524" layer="2"/>
+<via x="7.62" y="27.94" extent="1-16" drill="0.35"/>
+<wire x1="7.62" y1="25.654" x2="7.62" y2="27.94" width="0.1524" layer="1"/>
+<wire x1="7.62" y1="30.610925" x2="7.62" y2="27.94" width="0.1524" layer="2"/>
 </signal>
 <signal name="N$11">

Commit message: up
Parts:
- added DPOWER: DPOWER, pinhead:1X02
- GLORY: value 22-23-2021 -> GLORY
Connections:
- net GND: now also DPOWER.2
- net VCC: now also DPOWER.1
Routing:
- net VCC: track 222.3 -> 224.1 mm
- net GND: vias 20 -> 33
Changed lines of the file:
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@@
 <attribute name="VALUE" x="46.99" y="28.321" size="1.27" layer="27" ratio="10" rot="R180"/>
 </element>
-<element name="GLORY" library="con-molex" library_urn="urn:adsk.eagle:library:165" package="22-23-2021" package3d_urn="urn:adsk.eagle:package:8078633/1" value="22-23-2021" x="58.42" y="34.29" smashed="yes">
+<element name="GLORY" library="con-molex" library_urn="urn:adsk.eagle:library:165" package="22-23-2021" package3d_urn="urn:adsk.eagle:package:8078633/1" value="GLORY" x="58.42" y="34.29" smashed="yes">
 <attribute name="MF" value="MOLEX" x="58.42" y="34.29" size="1.778" layer="27" display="off"/>
 <attribute name="MPN" value="22-23-2021" x="58.42" y="34.29" size="1.778" layer="27" display="off"/>
@@
 <attribute name="POPULARITY" value="28" x="86.36" y="38.1" size="1.778" layer="27" display="off"/>
 <attribute name="VALUE" x="88.9" y="36.83" size="1.27" layer="27" rot="R90"/>
+</element>
+<element name="DPOWER" library="pinhead" library_urn="urn:adsk.eagle:library:325" package="1X02" package3d_urn="urn:adsk.eagle:package:22435/2" value="DPOWER" x="80.01" y="3.81" smashed="yes" rot="R180">
+<attribute name="NAME" x="82.6262" y="1.9812" size="1.27" layer="25" ratio="10" rot="R180"/>
+<attribute name="POPULARITY" value="98" x="80.01" y="3.81" size="1.778" layer="27" rot="R180" display="off"/>
+<attribute name="VALUE" x="82.55" y="6.985" size="1.27" layer="27" rot="R180"/>
 </element>
 </elements>
@@
 <wire x1="81.28" y1="39.8526" x2="86.2584" y2="39.8526" width="0.3048" layer="1"/>
 <wire x1="86.2584" y1="39.8526" x2="86.36" y2="39.85" width="0.3048" layer="1"/>
+<contactref element="DPOWER" pad="2"/>
+<via x="26.67" y="6.35" extent="1-16" drill="0.35"/>
+<via x="19.05" y="8.89" extent="1-16" drill="0.35"/>
+<via x="72.39" y="46.99" extent="1-16" drill="0.35"/>
+<via x="72.39" y="8.89" extent="1-16" drill="0.35"/>
+<via x="53.34" y="27.94" extent="1-16" drill="0.35"/>
+<via x="43.18" y="33.02" extent="1-16" drill="0.35"/>
+<via x="34.29" y="29.21" extent="1-16" drill="0.35"/>
+<via x="63.5" y="27.94" extent="1-16" drill="0.35"/>
+<via x="44.45" y="31.75" extent="1-16" drill="0.35"/>
+<via x="62.23" y="41.91" extent="1-16" drill="0.35"/>
+<via x="38.1" y="46.99" extent="1-16" drill="0.35"/>
+<via x="38.1" y="45.72" extent="1-16" drill="0.35"/>
+<via x="38.1" y="44.45" extent="1-16" drill="0.35"/>
 </signal>
 <signal name="VCC" class="1">
@@
 <wire x1="86.1822" y1="11.5062" x2="87.1728" y2="12.4968" width="0.3048" layer="2"/>
 <wire x1="86.1822" y1="10.9728" x2="86.1822" y2="11.5062" width="0.3048" layer="2"/>
-<wire x1="80.0862" y1="4.8768" x2="86.1822" y2="10.9728" width="0.3048" layer="2"/>
-<wire x1="59.2074" y1="4.8768" x2="80.0862" y2="4.8768" width="0.3048" layer="2"/>
 <wire x1="46.3296" y1="27.6606" x2="46.3296" y2="29.2608" width="0.3048" layer="1"/>
 <wire x1="46.3296" y1="26.289" x2="46.3296" y2="27.6606" width="0.3048" layer="2"/>
@@
 <wire x1="59.69" y1="34.29" x2="57.15" y2="34.29" width="0.3048" layer="1"/>
 <wire x1="53.3019" y1="38.1381" x2="57.15" y2="34.29" width="0.3048" layer="2"/>
+<contactref element="DPOWER" pad="1"/>
+<wire x1="81.3054" y1="6.096" x2="81.3054" y2="4.8768" width="0.3048" layer="2"/>
+<wire x1="81.3054" y1="4.8768" x2="81.3054" y2="3.81" width="0.3048" layer="2"/>
+<wire x1="86.1822" y1="10.9728" x2="81.3054" y2="6.096" width="0.3048" layer="2"/>
+<wire x1="81.3054" y1="3.81" x2="81.28" y2="3.81" width="0.3048" layer="2"/>
+<wire x1="59.2074" y1="4.8768" x2="81.3054" y2="4.8768" width="0.3048" layer="2"/>
 </signal>
 <signal name="N$1">
