File: touch.brd (EAGLE design)
At the start: 91.4 x 50.5 mm, 37 parts, among them IC1 MAX203ECWP, IC2 PIC18F14Q41-I_SO

Commit message: up
Parts:
- added PMOD: Pmod, con-lstb:MA06-2
Connections:
- net CS: now also PMOD.1
- net GND: now also PMOD.10, PMOD.9
- net MISC: now also PMOD.2
- net MISO: now also PMOD.5
- net MOSI: now also PMOD.3
- net RELAY: now also PMOD.4
- net SCK: now also PMOD.7
- net SMCLEAR: now also PMOD.6
- net TX1: now also PMOD.8
- net VCC: now also PMOD.11, PMOD.12
Routing:
- net SMCLEAR: track 79.5 -> 141.3 mm, vias 1 -> 2
- net RELAY: track 54.7 -> 106.6 mm
- net MISC: track 52.3 -> 103.3 mm, vias 1 -> 2
- net TX1: track 54.7 -> 90.8 mm
- net MOSI: track 49.1 -> 83.9 mm
- net CS: track 36.9 -> 69.6 mm
- net SCK: track 48.0 -> 76.3 mm
- net MISO: track 42.0 -> 66.8 mm
- net VCC: track 224.1 -> 232.2 mm
