File: touch.brd (EAGLE design)
At the start: 91.4 x 50.5 mm, 38 parts, among them IC1 MAX203ECWP, IC2 PIC18F14Q41-I_SO

Commit message: up
Parts:
- C1: value 10uf -> 0.1uf
- C2: value 0.1 -> 10uf
Routing:
- net GND: vias 33 -> 38
Other:
- board text added: "Q41 vtouch 1.3"
- board text removed: "Q41 vtouch 1.2"
Changed lines of the file:
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@@
 <hole x="87.63" y="3.81" drill="2.54"/>
 <hole x="87.63" y="46.99" drill="2.54"/>
-<text x="64.77" y="22.86" size="1.778" layer="1" font="vector" ratio="15" rot="R90">Q41 vtouch 1.2</text>
+<text x="64.77" y="22.86" size="1.778" layer="1" font="vector" ratio="15" rot="R90">Q41 vtouch 1.3</text>
 </plain>
 <attributes>
@@
 <attribute name="VALUE" x="7.62" y="24.0299" size="0.02" layer="27" rot="R90"/>
 </element>
-<element name="C1" library="rcl" library_urn="urn:adsk.eagle:library:334" package="C0805" package3d_urn="urn:adsk.eagle:package:23617/2" value="10uf" x="35.56" y="16.51" smashed="yes" rot="R90">
+<element name="C1" library="rcl" library_urn="urn:adsk.eagle:library:334" package="C0805" package3d_urn="urn:adsk.eagle:package:23617/2" value="0.1uf" x="35.56" y="16.51" smashed="yes" rot="R90">
 <attribute name="NAME" x="34.29" y="15.24" size="1.27" layer="25" rot="R90"/>
 <attribute name="POPULARITY" value="63" x="35.56" y="16.51" size="1.778" layer="27" rot="R90" display="off"/>
@@
 <attribute name="VALUE" x="36.83" y="19.05" size="1.27" layer="27" rot="R90"/>
 </element>
-<element name="C2" library="rcl" library_urn="urn:adsk.eagle:library:334" package="C0805" package3d_urn="urn:adsk.eagle:package:23617/2" value="0.1" x="31.75" y="16.51" smashed="yes" rot="R90">
+<element name="C2" library="rcl" library_urn="urn:adsk.eagle:library:334" package="C0805" package3d_urn="urn:adsk.eagle:package:23617/2" value="10uf" x="31.75" y="16.51" smashed="yes" rot="R90">
 <attribute name="NAME" x="30.48" y="15.24" size="1.27" layer="25" rot="R90"/>
 <attribute name="POPULARITY" value="63" x="31.75" y="16.51" size="1.778" layer="27" rot="R90" display="off"/>
@@
 <attribute name="MOUSER_PART_NUMBER" value="653-B3W-9000-Y1N" x="6.35" y="6.35" size="1.778" layer="27" display="off"/>
 <attribute name="MOUSER_PRICE-STOCK" value="https://www.mouser.com/Search/Refine.aspx?Keyword=653-B3W-9000-Y1N" x="6.35" y="6.35" size="1.778" layer="27" display="off"/>
-<attribute name="NAME" x="5.943009375" y="6.3067" size="1.27" layer="25" align="center"/>
+<attribute name="NAME" x="13.563009375" y="2.4967" size="1.27" layer="25" align="center"/>
 <attribute name="RS_PART_NUMBER" value="0492777P" x="6.35" y="6.35" size="1.778" layer="27" display="off"/>
 <attribute name="RS_PRICE-STOCK" value="http://uk.rs-online.com/web/p/products/0492777P" x="6.35" y="6.35" size="1.778" layer="27" display="off"/>
@@
 <attribute name="MF" value="" x="44.45" y="25.4" size="1.778" layer="27" rot="R180" display="off"/>
 <attribute name="MPN" value="" x="44.45" y="25.4" size="1.778" layer="27" rot="R180" display="off"/>
-<attribute name="NAME" x="50.8" y="23.749" size="1.27" layer="25" ratio="10" rot="R180"/>
+<attribute name="NAME" x="59.69" y="26.289" size="1.27" layer="25" ratio="10" rot="R180"/>
 <attribute name="OC_FARNELL" value="unknown" x="44.45" y="25.4" size="1.778" layer="27" rot="R180" display="off"/>
 <attribute name="OC_NEWARK" value="unknown" x="44.45" y="25.4" size="1.778" layer="27" rot="R180" display="off"/>
@@
 <contactref element="PMOD" pad="9"/>
 <contactref element="PMOD" pad="10"/>
+<via x="26.67" y="2.54" extent="1-16" drill="0.35"/>
+<polygon width="0.1524" layer="1">
+<vertex x="25.4" y="8.89"/>
+<vertex x="25.4" y="1.27"/>
+<vertex x="44.45" y="1.27"/>
+<vertex x="44.45" y="2.54"/>
+<vertex x="27.94" y="2.54"/>
+<vertex x="27.94" y="8.89"/>
+</polygon>
+<via x="27.94" y="19.05" extent="1-16" drill="0.35"/>
+<via x="30.48" y="29.21" extent="1-16" drill="0.35"/>
+<via x="45.72" y="5.08" extent="1-16" drill="0.35"/>
+<via x="53.34" y="41.91" extent="1-16" drill="0.35"/>
 </signal>
 <signal name="VCC" class="1">
