File: touch.sch (EAGLE design)
At the start: 25 parts, among them IC1 MAX203ECWP, IC2 PIC18F14Q41-I_SO, X1 22-23-2021

Commit message: up
Parts:
- added C7: 10uf, rcl:C-USC0805
- added F1: 0.75A, polyfuse-smd_10:1206L075SL
- added L1: 1000, inductor-neosid:SM-1206
- C1, C4: value (none) -> 10uf
- C2, C3, C5, C6: value (none) -> 0.1
- D1: value (none) -> 5.6V
- R1, R2: value (none) -> 56
- R3: value (none) -> 10K
- R4: value (none) -> 1k
- R5: value (none) -> 200
Connections:
- new net N$16: F1.2, X1-1.S
- new net N$20: F1.1, L1.1
- net GND: now also C7.2
- net VCC: now also C7.1, L1.2; no longer X1-1.S
Other:
- moved on the sheet: D1

Commit message: up
Parts:
- added LED_MODE: RED, led:LEDCHIPLED_0805
- added LED_POWER: GREEN, led:LEDCHIPLED_0805
- added R6, R7: 200, rcl:R-US_R0805
- added SV2: (no value), con-lstb:MA04-2
- added SV3: (no value), con-lstb:MA03-2
Connections:
- removed net N$17: C5.1, R2.1, R3.1, S1.1, S1.2
- new net CS: IC2.RB6, SV2.6
- new net MIN0: IC2.RC0, SV2.1
- new net MIN1: IC2.RC3, SV2.3
- new net MISC: IC2.RB7, SV3.3
- new net MISO: IC2.RB4, SV2.7
- new net MLED: IC2.RC4, R7.2
- new net MOSI: IC2.RA2, SV2.5
- new net N$21: LED_POWER.A, R6.1
- new net N$22: LED_MODE.A, R7.1
- new net RELAY: IC2.RC7, SV3.1
- new net RLED: IC2.RC5, R4.1
- new net SCK: IC2.RA4, SV2.8
- new net SMCLEAR: C5.1, R2.1, R3.1, S1.1, S1.2, SV3.5
- net GND: now also LED_MODE.C, LED_POWER.C, SV2.2, SV2.4, SV3.2
- net VCC: now also R6.2; no longer R4.1

Commit message: up
Parts:
- added TTLRS232: (no value), con-lstb:MA05-1
- renumbered SV1 to ICSP, SV2 to DIO2/SPI, SV3 to DIO3, X1 to POWER
Connections:
- net CLKIN: now also DIO3.4
- net GND: now also TTLRS232.1
- net RX1: now also TTLRS232.2
- net RX2: now also TTLRS232.4
- net TX1: now also TTLRS232.3
- net TX2: now also TTLRS232.5
- net VCC: now also DIO3.6

Commit message: up
Connections:
- net GND: now also HOST_PORT1.5, ICSP.3; no longer HOST_PORT1.1, ICSP.2
- net VCC: now also ICSP.2; no longer ICSP.3
Changed lines of the file:
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@@
 <part name="P+1" library="supply1" library_urn="urn:adsk.eagle:library:371" deviceset="VCC" device=""/>
 <part name="GND6" library="supply1" library_urn="urn:adsk.eagle:library:371" deviceset="GND" device=""/>
-<part name="GND7" library="supply1" library_urn="urn:adsk.eagle:library:371" deviceset="GND" device=""/>
 <part name="C1" library="rcl" library_urn="urn:adsk.eagle:library:334" deviceset="C-US" device="C0805" package3d_urn="urn:adsk.eagle:package:23617/2" value="10uf"/>
 <part name="C2" library="rcl" library_urn="urn:adsk.eagle:library:334" deviceset="C-US" device="C0805" package3d_urn="urn:adsk.eagle:package:23617/2" value="0.1"/>
@@
 <part name="GND10" library="supply1" library_urn="urn:adsk.eagle:library:371" deviceset="GND" device=""/>
 <part name="GND11" library="supply1" library_urn="urn:adsk.eagle:library:371" deviceset="GND" device=""/>
-<part name="GND12" library="supply1" library_urn="urn:adsk.eagle:library:371" deviceset="GND" device=""/>
-<part name="P+4" library="supply1" library_urn="urn:adsk.eagle:library:371" deviceset="VCC" device=""/>
 <part name="R1" library="rcl" library_urn="urn:adsk.eagle:library:334" deviceset="R-US_" device="R0805" package3d_urn="urn:adsk.eagle:package:23553/2" value="56"/>
 <part name="R2" library="rcl" library_urn="urn:adsk.eagle:library:334" deviceset="R-US_" device="R0805" package3d_urn="urn:adsk.eagle:package:23553/2" value="56"/>
@@
 <part name="TTLRS232" library="con-lstb" library_urn="urn:adsk.eagle:library:162" deviceset="MA05-1" device="" package3d_urn="urn:adsk.eagle:package:8332/1"/>
 <part name="GND22" library="supply1" library_urn="urn:adsk.eagle:library:371" deviceset="GND" device=""/>
+<part name="GND12" library="supply1" library_urn="urn:adsk.eagle:library:371" deviceset="GND" device=""/>
+<part name="P+4" library="supply1" library_urn="urn:adsk.eagle:library:371" deviceset="VCC" device=""/>
+<part name="GND23" library="supply1" library_urn="urn:adsk.eagle:library:371" deviceset="GND" device=""/>
 </parts>
 <sheets>
@@
 <attribute name="VALUE" x="193.04" y="68.58" size="1.778" layer="96" rot="R180"/>
 </instance>
-<instance part="GND7" gate="1" x="185.42" y="25.4" smashed="yes" rot="R90">
-<attribute name="VALUE" x="187.96" y="25.4" size="1.778" layer="96"/>
-</instance>
 <instance part="C1" gate="G$1" x="12.7" y="60.96" smashed="yes">
 <attribute name="NAME" x="13.716" y="61.595" size="1.778" layer="95"/>
@@
 <attribute name="VALUE" x="2.54" y="58.42" size="1.778" layer="96" rot="R270"/>
 </instance>
-<instance part="GND12" gate="1" x="58.42" y="5.08" smashed="yes">
-<attribute name="VALUE" x="55.88" y="2.54" size="1.778" layer="96"/>
-</instance>
-<instance part="P+4" gate="VCC" x="58.42" y="12.7" smashed="yes">
-<attribute name="VALUE" x="55.88" y="10.16" size="1.778" layer="96" rot="R90"/>
-</instance>
 <instance part="R1" gate="G$1" x="12.7" y="45.72" smashed="yes">
 <attribute name="NAME" x="8.89" y="47.2186" size="1.778" layer="95"/>
@@
 <instance part="GND22" gate="1" x="101.6" y="2.54" smashed="yes">
 <attribute name="VALUE" x="99.06" y="0" size="1.778" layer="96"/>
+</instance>
+<instance part="GND12" gate="1" x="60.96" y="10.16" smashed="yes" rot="R90">
+<attribute name="VALUE" x="63.5" y="7.62" size="1.778" layer="96" rot="R90"/>
+</instance>
+<instance part="P+4" gate="VCC" x="58.42" y="5.08" smashed="yes" rot="R180">
+<attribute name="VALUE" x="60.96" y="7.62" size="1.778" layer="96" rot="R270"/>
+</instance>
+<instance part="GND23" gate="1" x="170.18" y="25.4" smashed="yes" rot="R270">
+<attribute name="VALUE" x="167.64" y="25.4" size="1.778" layer="96" rot="R180"/>
 </instance>
 </instances>
@@
 <pinref part="GND6" gate="1" pin="GND"/>
 <junction x="182.88" y="68.58"/>
-</segment>
-<segment>
-<pinref part="HOST_PORT1" gate="G$1" pin="1"/>
-<pinref part="GND7" gate="1" pin="GND"/>
-<junction x="182.88" y="25.4"/>
 </segment>
 <segment>
@@
 </segment>
 <segment>
-<pinref part="ICSP" gate="1" pin="2"/>
-<wire x1="43.18" y1="-2.54" x2="43.18" y2="7.62" width="0.1524" layer="91"/>
-<wire x1="43.18" y1="7.62" x2="58.42" y2="7.62" width="0.1524" layer="91"/>
-<pinref part="GND12" gate="1" pin="GND"/>
-<junction x="43.18" y="-2.54"/>
-<junction x="58.42" y="7.62"/>
-</segment>
-<segment>
 <pinref part="C5" gate="G$1" pin="2"/>
 <pinref part="GND13" gate="1" pin="GND"/>
@@
 <pinref part="GND22" gate="1" pin="GND"/>
 <junction x="101.6" y="5.08"/>
+</segment>
+<segment>
+<pinref part="ICSP" gate="1" pin="3"/>
+<wire x1="40.64" y1="-2.54" x2="40.64" y2="10.16" width="0.1524" layer="91"/>
+<wire x1="40.64" y1="10.16" x2="58.42" y2="10.16" width="0.1524" layer="91"/>
+<junction x="40.64" y="-2.54"/>
+<pinref part="GND12" gate="1" pin="GND"/>
+<junction x="58.42" y="10.16"/>
+</segment>
+<segment>
+<pinref part="HOST_PORT1" gate="G$1" pin="5"/>
+<pinref part="GND23" gate="1" pin="GND"/>
+<junction x="172.72" y="25.4"/>
 </segment>
 </net>
@@
 </segment>
 <segment>
-<pinref part="ICSP" gate="1" pin="3"/>
-<wire x1="40.64" y1="-2.54" x2="40.64" y2="10.16" width="0.1524" layer="91"/>
-<wire x1="40.64" y1="10.16" x2="58.42" y2="10.16" width="0.1524" layer="91"/>
-<pinref part="P+4" gate="VCC" pin="VCC"/>
-<junction x="40.64" y="-2.54"/>
-<junction x="58.42" y="10.16"/>
-</segment>
-<segment>
 <pinref part="R3" gate="G$1" pin="2"/>
 <pinref part="P+5" gate="VCC" pin="VCC"/>
@@
 <junction x="134.62" y="-5.08"/>
 </segment>
+<segment>
+<pinref part="ICSP" gate="1" pin="2"/>
+<wire x1="43.18" y1="-2.54" x2="43.18" y2="7.62" width="0.1524" layer="91"/>
+<wire x1="43.18" y1="7.62" x2="58.42" y2="7.62" width="0.1524" layer="91"/>
+<junction x="43.18" y="-2.54"/>
+<pinref part="P+4" gate="VCC" pin="VCC"/>
+<junction x="58.42" y="7.62"/>
+</segment>
 </net>

Commit message: up
Parts:
- removed LED_MODE: RED, led:LEDCHIPLED_0805
- removed LED_POWER: GREEN, led:LEDCHIPLED_0805
- added GLORY: 22-23-2021, con-molex:22-23-2021
- added MODE, PWR: Green, led:LEDCHIPLED_1206
- R4: value 1k -> 1.2k
- R6, R7: value 200 -> 1.2k
Connections:
- net N$10 renamed DB1
- net N$13 renamed DB0
- net N$15 renamed PGM
- removed net N$22: LED_MODE.A, R7.1
- new net N$17: MODE.A, R7.1
- net GND: now also MODE.C, PWR.C; no longer LED_MODE.C, LED_POWER.C
- net N$21: now also PWR.A; no longer LED_POWER.A
- net VCC: now also GLORY-1.S, GLORY-2.S

Commit message: up
Parts:
- added DPOWER: DPOWER, pinhead:PINHD-1X2
- GLORY: value 22-23-2021 -> GLORY
Connections:
- net GND: now also DPOWER.2
- net VCC: now also DPOWER.1
Changed lines of the file:
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@@
 <part name="P+4" library="supply1" library_urn="urn:adsk.eagle:library:371" deviceset="VCC" device=""/>
 <part name="GND23" library="supply1" library_urn="urn:adsk.eagle:library:371" deviceset="GND" device=""/>
-<part name="GLORY" library="con-molex" library_urn="urn:adsk.eagle:library:165" deviceset="22-23-2021" device="" package3d_urn="urn:adsk.eagle:package:8078633/1"/>
+<part name="GLORY" library="con-molex" library_urn="urn:adsk.eagle:library:165" deviceset="22-23-2021" device="" package3d_urn="urn:adsk.eagle:package:8078633/1" value="GLORY"/>
 <part name="P+10" library="supply1" library_urn="urn:adsk.eagle:library:371" deviceset="VCC" device=""/>
 <part name="P+11" library="supply1" library_urn="urn:adsk.eagle:library:371" deviceset="VCC" device=""/>
 <part name="PWR" library="led" library_urn="urn:adsk.eagle:library:259" deviceset="LED" device="CHIPLED_1206" package3d_urn="urn:adsk.eagle:package:15823/2" value="Green"/>
 <part name="MODE" library="led" library_urn="urn:adsk.eagle:library:259" deviceset="LED" device="CHIPLED_1206" package3d_urn="urn:adsk.eagle:package:15823/2" value="Green"/>
+<part name="DPOWER" library="pinhead" library_urn="urn:adsk.eagle:library:325" deviceset="PINHD-1X2" device="" package3d_urn="urn:adsk.eagle:package:22435/2" value="DPOWER"/>
+<part name="GND7" library="supply1" library_urn="urn:adsk.eagle:library:371" deviceset="GND" device=""/>
+<part name="P+12" library="supply1" library_urn="urn:adsk.eagle:library:371" deviceset="VCC" device=""/>
 </parts>
 <sheets>
@@
 <attribute name="VALUE" x="15.875" y="84.328" size="1.778" layer="96" rot="R90"/>
 </instance>
+<instance part="DPOWER" gate="G$1" x="104.14" y="66.04" smashed="yes">
+<attribute name="NAME" x="97.79" y="71.755" size="1.778" layer="95"/>
+<attribute name="VALUE" x="97.79" y="60.96" size="1.778" layer="96"/>
+</instance>
+<instance part="GND7" gate="1" x="91.44" y="63.5" smashed="yes">
+<attribute name="VALUE" x="88.9" y="60.96" size="1.778" layer="96"/>
+</instance>
+<instance part="P+12" gate="VCC" x="91.44" y="71.12" smashed="yes">
+<attribute name="VALUE" x="88.9" y="71.12" size="1.778" layer="96" rot="R180"/>
+</instance>
 </instances>
 <busses>
@@
 <pinref part="GND23" gate="1" pin="GND"/>
 <junction x="172.72" y="25.4"/>
+</segment>
+<segment>
+<pinref part="DPOWER" gate="G$1" pin="2"/>
+<wire x1="101.6" y1="66.04" x2="99.06" y2="66.04" width="0.1524" layer="91"/>
+<pinref part="GND7" gate="1" pin="GND"/>
+<junction x="99.06" y="66.04"/>
+<wire x1="99.06" y1="66.04" x2="91.44" y2="66.04" width="0.1524" layer="91"/>
+<junction x="91.44" y="66.04"/>
 </segment>
 </net>
@@
 <junction x="119.38" y="5.08"/>
 </segment>
+<segment>
+<pinref part="DPOWER" gate="G$1" pin="1"/>
+<wire x1="101.6" y1="68.58" x2="99.06" y2="68.58" width="0.1524" layer="91"/>
+<pinref part="P+12" gate="VCC" pin="VCC"/>
+<junction x="99.06" y="68.58"/>
+<wire x1="99.06" y1="68.58" x2="91.44" y2="68.58" width="0.1524" layer="91"/>
+<junction x="91.44" y="68.58"/>
+</segment>
 </net>
