File: touch.sch (EAGLE design)
At the start: 37 parts, among them IC1 MAX203ECWP, IC2 PIC18F14Q41-I_SO

Commit message: up
Parts:
- added PMOD: Pmod, con-lstb:MA06-2
Connections:
- net CS: now also PMOD.1
- net GND: now also PMOD.10, PMOD.9
- net MISC: now also PMOD.2
- net MISO: now also PMOD.5
- net MOSI: now also PMOD.3
- net RELAY: now also PMOD.4
- net SCK: now also PMOD.7
- net SMCLEAR: now also PMOD.6
- net TX1: now also PMOD.8
- net VCC: now also PMOD.11, PMOD.12
Changed lines of the file:
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@@
 <?xml version="1.0" encoding="utf-8"?>
 <!DOCTYPE eagle SYSTEM "eagle.dtd">
-<eagle version="9.7.0">
+<eagle version="9.6.2">
 <drawing>
 <settings>
@@
 <part name="GND7" library="supply1" library_urn="urn:adsk.eagle:library:371" deviceset="GND" device=""/>
 <part name="P+12" library="supply1" library_urn="urn:adsk.eagle:library:371" deviceset="VCC" device=""/>
+<part name="PMOD" library="con-lstb" library_urn="urn:adsk.eagle:library:162" deviceset="MA06-2" device="" package3d_urn="urn:adsk.eagle:package:8342/1" value="Pmod"/>
+<part name="GND24" library="supply1" library_urn="urn:adsk.eagle:library:371" deviceset="GND" device=""/>
+<part name="P+13" library="supply1" library_urn="urn:adsk.eagle:library:371" deviceset="VCC" device=""/>
+<part name="P+14" library="supply1" library_urn="urn:adsk.eagle:library:371" deviceset="VCC" device=""/>
+<part name="GND25" library="supply1" library_urn="urn:adsk.eagle:library:371" deviceset="GND" device=""/>
 </parts>
 <sheets>
@@
 <attribute name="VALUE" x="88.9" y="71.12" size="1.778" layer="96" rot="R180"/>
 </instance>
+<instance part="PMOD" gate="1" x="104.14" y="111.76" smashed="yes">
+<attribute name="VALUE" x="100.33" y="99.06" size="1.778" layer="96"/>
+<attribute name="NAME" x="100.33" y="120.142" size="1.778" layer="95"/>
+</instance>
+<instance part="GND24" gate="1" x="114.3" y="114.3" smashed="yes" rot="R90">
+<attribute name="VALUE" x="116.84" y="111.76" size="1.778" layer="96" rot="R90"/>
+</instance>
+<instance part="P+13" gate="VCC" x="111.76" y="119.38" smashed="yes">
+<attribute name="VALUE" x="109.22" y="119.38" size="1.778" layer="96" rot="R180"/>
+</instance>
+<instance part="P+14" gate="VCC" x="96.52" y="119.38" smashed="yes">
+<attribute name="VALUE" x="93.98" y="119.38" size="1.778" layer="96" rot="R180"/>
+</instance>
+<instance part="GND25" gate="1" x="93.98" y="114.3" smashed="yes" rot="R270">
+<attribute name="VALUE" x="91.44" y="116.84" size="1.778" layer="96" rot="R270"/>
+</instance>
 </instances>
 <busses>
@@
 <wire x1="99.06" y1="66.04" x2="91.44" y2="66.04" width="0.1524" layer="91"/>
 <junction x="91.44" y="66.04"/>
+</segment>
+<segment>
+<pinref part="PMOD" gate="1" pin="9"/>
+<pinref part="GND24" gate="1" pin="GND"/>
+</segment>
+<segment>
+<pinref part="PMOD" gate="1" pin="10"/>
+<pinref part="GND25" gate="1" pin="GND"/>
+<junction x="96.52" y="114.3"/>
 </segment>
 </net>
@@
 <wire x1="99.06" y1="68.58" x2="91.44" y2="68.58" width="0.1524" layer="91"/>
 <junction x="91.44" y="68.58"/>
+</segment>
+<segment>
+<pinref part="PMOD" gate="1" pin="11"/>
+<pinref part="P+13" gate="VCC" pin="VCC"/>
+<junction x="111.76" y="116.84"/>
+</segment>
+<segment>
+<pinref part="PMOD" gate="1" pin="12"/>
+<pinref part="P+14" gate="VCC" pin="VCC"/>
+<junction x="96.52" y="116.84"/>
 </segment>
 </net>
@@
 <label x="104.14" y="10.16" size="1.778" layer="95"/>
 </segment>
+<segment>
+<wire x1="96.52" y1="111.76" x2="93.98" y2="111.76" width="0.1524" layer="91"/>
+<pinref part="PMOD" gate="1" pin="8"/>
+<label x="78.74" y="111.76" size="1.778" layer="95"/>
+<junction x="96.52" y="111.76"/>
+<junction x="93.98" y="111.76"/>
+</segment>
 </net>
 <net name="RX1" class="0">
@@
 <label x="152.4" y="-2.54" size="1.778" layer="95"/>
 </segment>
+<segment>
+<wire x1="96.52" y1="109.22" x2="88.9" y2="109.22" width="0.1524" layer="91"/>
+<pinref part="PMOD" gate="1" pin="6"/>
+<junction x="96.52" y="109.22"/>
+<label x="78.74" y="109.22" size="1.778" layer="95"/>
+<junction x="88.9" y="109.22"/>
+</segment>
 </net>
 <net name="N$18" class="0">
@@
 <label x="152.4" y="-12.7" size="1.778" layer="95"/>
 </segment>
+<segment>
+<wire x1="96.52" y1="106.68" x2="93.98" y2="106.68" width="0.1524" layer="91"/>
+<pinref part="PMOD" gate="1" pin="4"/>
+<junction x="96.52" y="106.68"/>
+<label x="78.74" y="106.68" size="1.778" layer="95"/>
+<junction x="93.98" y="106.68"/>
+</segment>
 </net>
 <net name="MIN1" class="0">
@@
 <junction x="119.38" y="93.98"/>
 </segment>
+<segment>
+<wire x1="114.3" y1="111.76" x2="111.76" y2="111.76" width="0.1524" layer="91"/>
+<pinref part="PMOD" gate="1" pin="7"/>
+<junction x="111.76" y="111.76"/>
+<label x="119.38" y="111.76" size="1.778" layer="95"/>
+<junction x="114.3" y="111.76"/>
+</segment>
 </net>
 <net name="MOSI" class="0">
@@
 <junction x="142.24" y="91.44"/>
 </segment>
+<segment>
+<wire x1="111.76" y1="106.68" x2="116.84" y2="106.68" width="0.1524" layer="91"/>
+<pinref part="PMOD" gate="1" pin="3"/>
+<junction x="111.76" y="106.68"/>
+<label x="116.84" y="106.68" size="1.778" layer="95"/>
+<junction x="116.84" y="106.68"/>
+</segment>
 </net>
 <net name="MISO" class="0">
@@
 <junction x="147.32" y="93.98"/>
 </segment>
+<segment>
+<wire x1="111.76" y1="109.22" x2="121.92" y2="109.22" width="0.1524" layer="91"/>
+<pinref part="PMOD" gate="1" pin="5"/>
+<junction x="111.76" y="109.22"/>
+<junction x="121.92" y="109.22"/>
+<label x="124.46" y="109.22" size="1.778" layer="95"/>
+</segment>
 </net>
 <net name="CS" class="0">
@@
 <junction x="111.76" y="91.44"/>
 </segment>
+<segment>
+<wire x1="111.76" y1="104.14" x2="121.92" y2="104.14" width="0.1524" layer="91"/>
+<pinref part="PMOD" gate="1" pin="1"/>
+<junction x="111.76" y="104.14"/>
+<label x="121.92" y="104.14" size="1.778" layer="95"/>
+<junction x="121.92" y="104.14"/>
+</segment>
 </net>
 <net name="MISC" class="0">
@@
 <label x="154.94" y="-7.62" size="1.778" layer="95"/>
 </segment>
-</net>
+<segment>
+<wire x1="96.52" y1="104.14" x2="88.9" y2="104.14" width="0.1524" layer="91"/>
+<pinref part="PMOD" gate="1" pin="2"/>
+<junction x="96.52" y="104.14"/>
+<label x="78.74" y="104.14" size="1.778" layer="95"/>
+<junction x="88.9" y="104.14"/>
+</segment>
+</net>

Commit message: up
Parts:
- C1: value 10uf -> 0.1uf
- C2: value 0.1 -> 10uf
Changed lines of the file:
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@@
 <part name="P+1" library="supply1" library_urn="urn:adsk.eagle:library:371" deviceset="VCC" device=""/>
 <part name="GND6" library="supply1" library_urn="urn:adsk.eagle:library:371" deviceset="GND" device=""/>
-<part name="C1" library="rcl" library_urn="urn:adsk.eagle:library:334" deviceset="C-US" device="C0805" package3d_urn="urn:adsk.eagle:package:23617/2" value="10uf"/>
-<part name="C2" library="rcl" library_urn="urn:adsk.eagle:library:334" deviceset="C-US" device="C0805" package3d_urn="urn:adsk.eagle:package:23617/2" value="0.1"/>
+<part name="C1" library="rcl" library_urn="urn:adsk.eagle:library:334" deviceset="C-US" device="C0805" package3d_urn="urn:adsk.eagle:package:23617/2" value="0.1uf"/>
+<part name="C2" library="rcl" library_urn="urn:adsk.eagle:library:334" deviceset="C-US" device="C0805" package3d_urn="urn:adsk.eagle:package:23617/2" value="10uf"/>
 <part name="C3" library="rcl" library_urn="urn:adsk.eagle:library:334" deviceset="C-US" device="C0805" package3d_urn="urn:adsk.eagle:package:23617/2" value="0.1"/>
 <part name="C4" library="rcl" library_urn="urn:adsk.eagle:library:334" deviceset="C-US" device="C0805" package3d_urn="urn:adsk.eagle:package:23617/2" value="10uf"/>
